File: kicad/dimmer_or_current_regulator.kicad_sch (KiCad schematic)
At the start: 6 parts, among them Q1 MAC97A6

Commit message: update names
Parts:
- renumbered RC to R1, RV to VR1
Changed lines of the file:
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@@
   (symbol (lib_id "Device:R_Variable") (at 110.49 45.72 90) (unit 1)
     (in_bom yes) (on_board yes) (fields_autoplaced)
-    (property "Reference" "RV" (id 0) (at 110.49 38.1 90))
+    (property "Reference" "VR1" (id 0) (at 110.49 38.1 90))
     (property "Value" "R_Variable" (id 1) (at 110.49 40.64 90))
     (property "Footprint" "" (id 2) (at 110.49 47.498 90)
@@
   (symbol (lib_id "Device:R") (at 125.73 45.72 90) (unit 1)
     (in_bom yes) (on_board yes) (fields_autoplaced)
-    (property "Reference" "RC" (id 0) (at 125.73 39.37 90))
+    (property "Reference" "R1" (id 0) (at 125.73 39.37 90))
     (property "Value" "R" (id 1) (at 125.73 41.91 90))
     (property "Footprint" "" (id 2) (at 125.73 47.498 90)
@@
     )
     (path "/cce26f28-0607-44b7-b6e6-6ff618b1d62d"
-      (reference "RC") (unit 1) (value "R") (footprint "")
+      (reference "R1") (unit 1) (value "R") (footprint "")
     )
     (path "/f47b4270-1cf8-499b-9a05-0ef4b62bb7ea"
@@
     )
     (path "/1fbdff44-7ee7-44a1-af4d-b8965b2e170b"
-      (reference "RV") (unit 1) (value "R_Variable") (footprint "")
+      (reference "VR1") (unit 1) (value "R_Variable") (footprint "")
     )
   )
